File: kicad/power.kicad_sch (KiCad schematic)
At the start: 20 parts, among them U19 74LS07, U3 74LS27, U32 74S20, U4 74S04, U43 74LS74, U44 74S74, U45 74LS04, U59 74LS00, U6 74LS00, U60 74LS10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

Commit message: finalized schematic
Parts:
- removed U19: 74LS07, Package_DIP:DIP-14_W7.62mm, symbol 74xx:74LS07
- removed U3: 74LS27, symbol 74xx:74LS27
- removed U32: 74S20, symbol 74xx:74LS20
- removed U4: 74S04, symbol 74xx:74LS04
- removed U43, U76: 74LS74, Package_DIP:DIP-14_W7.62mm, symbol 74xx:74LS74
- removed U44: 74S74, symbol 74xx:74LS74
- removed U45, U73: 74LS04, Package_DIP:DIP-14_W7.62mm, symbol 74xx:74LS04
- removed U59, U90: 74LS00, Package_DIP:DIP-14_W7.62mm, symbol 74xx:74LS00
- removed U6: 74LS00, symbol 74xx:74LS00
- removed U60: 74LS10, Package_DIP:DIP-14_W7.62mm, symbol 74xx:74LS10
- removed U61: 74LS14, Package_DIP:DIP-14_W7.62mm, symbol 74xx:74LS14
- removed U72, U87: 74S08, Package_DIP:DIP-14_W7.62mm, symbol 74xx:74LS08
- removed U75: 74LS32, Package_DIP:DIP-14_W7.62mm, symbol 74xx:74LS32
- removed U77: 74LS08, Package_DIP:DIP-14_W7.62mm, symbol 74xx:74LS08
- removed U92: 74S10, Package_DIP:DIP-14_W7.62mm, symbol 74xx:74LS10
- removed U93: 74S74, Package_DIP:DIP-14_W7.62mm, symbol 74xx:74LS74
