File: kicad/xl-7.kicad_sch (KiCad schematic)
At the start: 51 parts, among them J10 Keylock, J11 Speaker, J12 Turbo LED, J13 Reset switch, J9 Keyboard, Q1 BC547, SW1 Turbo switch, SW2 XT CONFIG, U19 74LS07, U20 74LS175, U30 74LS322, U31 PAL R6, U32 74S20, U4 74S04, U43 74LS74, U44 74S74, U45 74LS04, U59 74LS00, U6 74LS00, U60 74LS10, U61 74LS14, U72 74S08, U73 74LS04, U74 74LS138, U75 74LS32, U76 74LS74, U77 74LS08, U90 74LS00, U92 74S10, U93 74S74, Y2 24M

Commit message: finalized schematic
Parts:
- removed U31: PAL R6, symbol 74xx:74LS322
- removed U32: 74S20, symbol 74xx:74LS20
- removed U44: 74S74, symbol 74xx:74LS74
- removed U45: 74LS04, Package_DIP:DIP-14_W7.62mm, symbol 74xx:74LS04
- removed U59: 74LS00, Package_DIP:DIP-14_W7.62mm, symbol 74xx:74LS00
- removed unit 4 of U6
- removed U60: 74LS10, Package_DIP:DIP-14_W7.62mm, symbol 74xx:74LS10
- removed unit 1 of U61
- removed unit 2 of U61
- removed unit 3 of U61
- removed unit 2 of U72
- removed unit 1 of U73
- removed unit 5 of U73
- removed U74: 74LS138, Package_DIP:DIP-16_W7.62mm, symbol 74xx:74LS138
- removed U75: 74LS32, Package_DIP:DIP-14_W7.62mm, symbol 74xx:74LS32
- removed U76: 74LS74, Package_DIP:DIP-14_W7.62mm, symbol 74xx:74LS74
- removed U77: 74LS08, Package_DIP:DIP-14_W7.62mm, symbol 74xx:74LS08
- removed U92: 74S10, Package_DIP:DIP-14_W7.62mm, symbol 74xx:74LS10
- removed unit 1 of U93
- added unit 7 of U19
- added U3: 74LS27, symbol 74xx:74LS27
- added U32: 74S20, symbol 74xx:74LS20
- added unit 7 of U4
- added unit 3 of U43
- added U44: 74S74, symbol 74xx:74LS74
- added U45: 74LS04, Package_DIP:DIP-14_W7.62mm, symbol 74xx:74LS04
- added U59: 74LS00, Package_DIP:DIP-14_W7.62mm, symbol 74xx:74LS00
- added unit 5 of U6
- added U60: 74LS10, Package_DIP:DIP-14_W7.62mm, symbol 74xx:74LS10
- added unit 7 of U61
- added unit 5 of U72
- added unit 7 of U73
- added U75: 74LS32, Package_DIP:DIP-14_W7.62mm, symbol 74xx:74LS32
- added U76: 74LS74, Package_DIP:DIP-14_W7.62mm, symbol 74xx:74LS74
- added U77: 74LS08, Package_DIP:DIP-14_W7.62mm, symbol 74xx:74LS08
- added U87: 74S08, Package_DIP:DIP-14_W7.62mm, symbol 74xx:74LS08
- added unit 5 of U90
- added U92: 74S10, Package_DIP:DIP-14_W7.62mm, symbol 74xx:74LS10
- added unit 3 of U93
Connections:
- net L2 is gone; now on net VCC: U30.8 (OE), U43.12 (D)
- net L3 is gone; now on net KBD: U19.1, U30.1 (G), U43.10 (~{S}), U43.8 (~{Q})
- net GND: now also U19.7 (GND), U3.7 (GND), U32.7 (GND), U4.7 (GND), U43.7 (GND), U44.7 (GND), U45.7 (GND), U59.7 (GND), U6.7 (GND), U60.7 (GND), U61.7 (GND), U72.7 (GND), U73.7 (GND), U75.7 (GND), U76.7 (GND), U77.7 (GND), U87.7 (GND), U90.7 (GND), U92.7 (GND), U93.7 (GND)
- net KBC: now also R3.2
- net KBD: now also R2.2
- net RESDRV: now also R4.2
- net VCC: now also R2.1, R3.1, R4.1, RP1.1 (common), RP3.1 (common), U19.14 (VCC), U3.14 (VCC), U32.14 (VCC), U4.14 (VCC), U43.14 (VCC), U44.14 (VCC), U45.14 (VCC), U59.14 (VCC), U6.14 (VCC), U60.14 (VCC), U61.14 (VCC), U72.14 (VCC), U73.14 (VCC), U75.14 (VCC), U76.14 (VCC), U77.14 (VCC), U87.14 (VCC), U90.14 (VCC), U92.14 (VCC), U93.14 (VCC)
- net at C1.2, Y2.1: now also R8.1
- net U92: now reaches RP3.10 (R9)
- net IORDY: now reaches RP3.2 (R1)
- net XIOW: now reaches RP3.3 (R2)
- net IOCHK: now reaches RP3.7 (R6)
- net EOP: now reaches RP3.8 (R7)
- net MWT: now reaches RP1.10 (R9)
- net XIOR: now reaches RP1.2 (R1)
- net XMEMR: now reaches RP1.3 (R2)
- net RESRVD: now reaches RP1.4 (R3)
- net MEMR: now reaches RP1.5 (R4)
- net INTA: now reaches RP1.6 (R5)
- net MEMW: now reaches RP1.7 (R6)
- net IOR: now reaches RP1.8 (R7)
- net IOW: now reaches RP1.9 (R8)
- no-connect marks 8 -> 30
Other:
- removed sheet Power
- moved on the sheet: C1, J10, J11, J9, Q1, R10, R2, R20, R22, R23, R3, R4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
